File: KiCad/QudrupedTurret.kicad_sch (KiCad schematic)
At the start: 16 parts, among them M1 Base_Servo_Front_Right, M10 Reloading_Servo, M11 Flywheel_Motor_Left, M12 Flywheel_Motor_Right, M2 Base_Servo_Front_Left, M3 Base_Servo_Back_Left, M4 Base_Servo_Back_Right, M5 Knee_Servo_Front_Right, M6 Knee_Servo_Front_Left, M7 Knee_Servo_Back_Left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

Commit message: Updated Wiring Schematic
Parts:
- U1: symbol RF_Controller:ESP32_DevKitC_30 -> DevBoards:ESP32_DevKitC_30
Connections:
- no-connect marks 0 -> 15
Other:
- moved on the sheet: BT1, M1, M10, M11, M12, M2, M3, M4, M5, M6, M7, M8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
